File: osvitovka_pcb/osvitovka/vrtackaRamku4m/vrtackaRamku4m.kicad_pcb (KiCad board)
At the start: 2 copper layers, 24 parts, among them J1 Screw_Terminal_01x01, J3 Screw_Terminal_01x01, J5 M+, J6 M-, Q1 BUZ11, SW1 SW_Push, U1 LM78M05_TO220, U2 LTV-817S

Commit message: Finální PCB k vytisknutí.
Parts:
- removed the REF** at (63.5, 127.0)
- removed the REF** at (127.0, 127.0)
- removed the REF** at (127.0, 190.5)
- removed the REF** at (63.5, 190.5)
- added REF**: MountingHole_3.5mm_Pad, MountingHole:MountingHole_3.5mm_Pad, F.Cu at (108.0, 124.5)
- added REF**: MountingHole_3.5mm_Pad, MountingHole:MountingHole_3.5mm_Pad, F.Cu at (174.0, 124.5)
- added REF**: MountingHole_3.5mm_Pad, MountingHole:MountingHole_3.5mm_Pad, F.Cu at (174.0, 48.3)
- added REF**: MountingHole_3.5mm_Pad, MountingHole:MountingHole_3.5mm_Pad, F.Cu at (108.0, 48.3)
- moved R2 105.6 mm to (134.6, 73.7), turned to 270 degrees
- moved J6 105.4 mm to (142.2, 57.1), turned to 270 degrees
- moved SW1 101.6 mm to (138.4, 83.8), turned to 0 degrees
- moved U2 99.2 mm to (125.7, 73.7), turned to 90 degrees
- moved R1 98.3 mm to (139.7, 73.7), turned to 90 degrees
- moved R3 97.1 mm to (147.3, 97.8)
- moved R4 97.1 mm to (147.3, 100.3)
- moved R5 97.1 mm to (147.3, 95.2)
- moved HC-SR4 96.2 mm to (165.1, 57.1)
- moved DLed2 96.1 mm to (138.4, 104.1)
- moved A1 95.3 mm to (153.7, 69.8)
- moved D1 90.3 mm to (130.8, 61.0), turned to 0 degrees
- moved J3 89.9 mm to (143.5, 116.8)
- moved Q1 89.4 mm to (134.6, 68.6), turned to 0 degrees
- moved DLed1 86.2 mm to (130.8, 104.1)
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Connections:
- A1 pad 1: Net-(A1-Pad1) -> PWM1
- A1 pad 11: Net-(A1-Pad11) -> Btn1
- A1 pad 12: Btn1 -> Led_yellow
- A1 pad 13: Led_yellow -> Led_green
- A1 pad 14: Led_green -> Net-(A1-Pad14)
- A1 pad 5: PWM1 -> Net-(A1-Pad5)
- A1 pad 6: Net-(A1-Pad6) -> Trig
- A1 pad 7: Trig -> Echo
- A1 pad 8: Echo -> Net-(A1-Pad8)
Routing:
- net GND: track 228.6 -> 354.0 mm
- net +5V: track 102.5 -> 148.2 mm
- net +12V: track 184.2 -> 151.3 mm
- net Net-(Q1-Pad1): track 35.7 -> 11.3 mm
- net Net-(R1-Pad1): track 0.00 -> 20.0 mm
- net Net-(D1-Pad2): track 16.7 -> 35.5 mm
- net Btn1: track 29.1 -> 21.0 mm
- net PWM1: track 7.18 -> 14.9 mm
- net Net-(DLed1-Pad2): track 10.8 -> 18.4 mm
- net Trig: track 33.0 -> 31.0 mm
- net Echo: track 38.1 -> 36.1 mm
- net Net-(DLed2-Pad2): track 7.71 -> 8.24 mm
- added copper zone on F.Cu, net GND
Other:
- board text added: "+12V"
- board text added: "+5V"
- board text added: "Echo"
- board text added: "GND"
- board text added: "M+"
- board text added: "M-"
- board text added: "Trig"
