File: osvitovka_pcb/osvitovka/vrtackaRamku4m/vrtackaRamku4m.sch (KiCad schematic (older format))
At the start: 29 parts, among them J1 Screw_Terminal_01x01, J2 Screw_Terminal_01x01, J3 Screw_Terminal_01x01, J4 Screw_Terminal_01x01, J5 M+, J6 M-, J7 M+, J8 M-, Q1 BUZ11, Q2 BUZ11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

Commit message: Finální verze po OK CRC kontrole schématu.
Parts:
- renumbered R5 to R6, R6 to R7
Connections:
- wire segments 76 -> 78
Changed lines of the file:
@@
-$EndComp
-$Comp
-L power:+12V #PWR0105
-U 1 1 5FC93B8F
-P 1400 950
-F 0 "#PWR0105" H 1400 800 50  0001 C CNN
-F 1 "+12V" V 1415 1078 50  0000 L CNN
-F 2 "" H 1400 950 50  0001 C CNN
-F 3 "" H 1400 950 50  0001 C CNN
-	1    1400 950
-	0    1    1    0
 $EndComp
 $Comp
@@
 $EndComp
 $Comp
-L power:GND #PWR0107
-U 1 1 5FC95104
-P 2400 950
-F 0 "#PWR0107" H 2400 700 50  0001 C CNN
-F 1 "GND" V 2405 822 50  0000 R CNN
-F 2 "" H 2400 950 50  0001 C CNN
-F 3 "" H 2400 950 50  0001 C CNN
-	1    2400 950
-	0    -1   -1   0
-$EndComp
-Wire Wire Line
-	1250 950  1400 950
-Wire Wire Line
-	1250 1300 1400 1300
-Wire Wire Line
-	2250 950  2400 950
-Wire Wire Line
-	2250 1300 2400 1300
-$Comp
 L power:GND #PWR0108
 U 1 1 5FC95D7A
@@
 	1    0    0    -1
 $EndComp
-Wire Wire Line
-	9550 4050 9550 4200
-Wire Wire Line
-	9650 4050 9650 4200
 $Comp
 L power:+5V #PWR0110
@@
 	1    0    0    -1
 $EndComp
-Wire Wire Line
-	9450 1850 9450 2050
 NoConn ~ 9650 2050
 NoConn ~ 9750 2050
@@
 	1    0    0    -1
 $EndComp
-Wire Wire Line
-	5650 2850 5650 2950
 $Comp
 L power:GND #PWR0116
@@
 Wire Wire Line
 	4950 2350 4800 2350
-Wire Wire Line
-	4800 2350 4800 2950
 $Comp
 L Device:R R1
@@
 Wire Wire Line
 	6050 2150 6050 2100
-Wire Wire Line
-	6050 2550 6050 2950
 Wire Wire Line
 	6050 1600 6050 1650
@@
 	1900 4600 2100 4600
 Wire Wire Line
-	2400 4600 2600 4600
-Wire Wire Line
 	1400 5050 1600 5050
 Wire Wire Line
 	1900 5050 2100 5050
-Wire Wire Line
-	2400 5050 2600 5050
 Text GLabel 8900 3450 0    50   Input ~ 0
 Led_yellow
@@
 	0    -1   -1   0
 $EndComp
-Wire Wire Line
-	1100 5550 1550 5550
 Text GLabel 2500 5550 2    50   Input ~ 0
 Btn1
@@
 	0    1    1    0
 $EndComp
-Wire Wire Line
-	2400 5900 2600 5900
 Wire Wire Line
 	2100 5900 2000 5900
@@
 Wire Wire Line
 	1250 3600 1400 3600
-Wire Wire Line
-	5700 1600 5700 2150
 $Comp
 L Connector:Screw_Terminal_01x01 J5
@@
 	1    0    0    -1
 $EndComp
-Wire Wire Line
-	1500 2900 1500 2700
 $Comp
 L Isolator:LTV-817S U3
@@
 $EndComp
 $Comp
-L power:+12V #PWR?
+L power:+12V #PWR0122
 U 1 1 5FCE20A3
 P 5700 3700
-F 0 "#PWR?" H 5700 3550 50  0001 C CNN
+F 0 "#PWR0122" H 5700 3550 50  0001 C CNN
 F 1 "+12V" H 5715 3873 50  0000 C CNN
 F 2 "" H 5700 3700 50  0001 C CNN
@@
 $EndComp
 $Comp
-L Device:R R6
+L Device:R R7
 U 1 1 5FCE20A9
 P 5650 4800
-F 0 "R6" H 5720 4846 50  0000 L CNN
+F 0 "R7" H 5720 4846 50  0000 L CNN
 F 1 "10k" H 5720 4755 50  0000 L CNN
 F 2 "" V 5580 4800 50  0001 C CNN
@@
 	5650 4450 5750 4450
 $Comp
-L power:GND #PWR?
+L power:GND #PWR0123
 U 1 1 5FCE20B4
 P 5650 5050
-F 0 "#PWR?" H 5650 4800 50  0001 C CNN
+F 0 "#PWR0123" H 5650 4800 50  0001 C CNN
 F 1 "GND" H 5655 4877 50  0000 C CNN
 F 2 "" H 5650 5050 50  0001 C CNN
@@
 $EndComp
 $Comp
-L power:GND #PWR?
+L power:GND #PWR0124
 U 1 1 5FCE20BA
 P 6050 5050
-F 0 "#PWR?" H 6050 4800 50  0001 C CNN
+F 0 "#PWR0124" H 6050 4800 50  0001 C CNN
 F 1 "GND" H 6055 4877 50  0000 C CNN
 F 2 "" H 6050 5050 50  0001 C CNN
@@
 	1    0    0    -1
 $EndComp
-Wire Wire Line
-	5650 4950 5650 5050
-$Comp
-L power:GND #PWR?
+$Comp
+L power:GND #PWR0125
 U 1 1 5FCE20C1
 P 4800 5050
-F 0 "#PWR?" H 4800 4800 50  0001 C CNN
+F 0 "#PWR0125" H 4800 4800 50  0001 C CNN
 F 1 "GND" H 4805 4877 50  0000 C CNN
 F 2 "" H 4800 5050 50  0001 C CNN
@@
 Wire Wire Line
 	4950 4450 4800 4450
-Wire Wire Line
-	4800 4450 4800 5050
-$Comp
-L Device:R R5
+$Comp
+L Device:R R6
 U 1 1 5FCE20C9
 P 4650 4250
-F 0 "R5" V 4443 4250 50  0000 C CNN
+F 0 "R6" V 4443 4250 50  0000 C CNN
 F 1 "470" V 4534 4250 50  0000 C CNN
 F 2 "" V 4580 4250 50  0001 C CNN
@@
 	4200 4250 4500 4250
 $Comp
-L power:+12V #PWR?
+L power:+12V #PWR0126
 U 1 1 5FCE20D2
 P 6050 3700
-F 0 "#PWR?" H 6050 3550 50  0001 C CNN
+F 0 "#PWR0126" H 6050 3550 50  0001 C CNN
 F 1 "+12V" H 6065 3873 50  0000 C CNN
 F 2 "" H 6050 3700 50  0001 C CNN
@@
 	6050 4250 6050 4200
 Wire Wire Line
-	6050 4650 6050 5050
-Wire Wire Line
 	6050 3700 6050 3750
 Wire Wire Line
@@
 	6050 4200 6050 4150
 NoConn ~ 6350 5050
-Wire Wire Line
-	5700 3700 5700 4250
 $Comp
 L Connector:Screw_Terminal_01x01 J7
@@
 Wire Wire Line
 	8900 2750 9050 2750
+$Comp
+L power:+12V #PWR0105
+U 1 1 5FCF4A8C
+P 1400 950
+F 0 "#PWR0105" H 1400 800 50  0001 C CNN
+F 1 "+12V" V 1415 1078 50  0000 L CNN
+F 2 "" H 1400 950 50  0001 C CNN
+F 3 "" H 1400 950 50  0001 C CNN
+	1    1400 950
+	0    1    1    0
+$EndComp
+$Comp
+L power:GND #PWR0107
+U 1 1 5FCF4D70
+P 2400 950
+F 0 "#PWR0107" H 2400 700 50  0001 C CNN
+F 1 "GND" V 2405 822 50  0000 R CNN
+F 2 "" H 2400 950 50  0001 C CNN
+F 3 "" H 2400 950 50  0001 C CNN
+	1    2400 950
+	0    -1   -1   0
+$EndComp
+Wire Wire Line
+	2250 950  2300 950
+Wire Wire Line
+	1250 950  1300 950
+$Comp
+L power:PWR_FLAG #FLG0101
+U 1 1 5FCF95CF
+P 1300 950
+F 0 "#FLG0101" H 1300 1025 50  0001 C CNN
+F 1 "PWR_FLAG" H 1300 1123 50  0000 C CNN
+F 2 "" H 1300 950 50  0001 C CNN
+F 3 "~" H 1300 950 50  0001 C CNN
+	1    1300 950
+	1    0    0    -1
+$EndComp
+Connection ~ 1300 950
+Wire Wire Line
+	1300 950  1400 950
+$Comp
+L power:PWR_FLAG #FLG0104
+U 1 1 5FCFAF58
+P 2300 950
+F 0 "#FLG0104" H 2300 1025 50  0001 C CNN
+F 1 "PWR_FLAG" H 2300 1123 50  0000 C CNN
+F 2 "" H 2300 950 50  0001 C CNN
+F 3 "~" H 2300 950 50  0001 C CNN
+	1    2300 950
+	1    0    0    -1
+$EndComp
+Connection ~ 2300 950
+Wire Wire Line
+	2300 950  2400 950
+Wire Wire Line
+	2400 4600 2600 4600
+Wire Wire Line
+	2400 5050 2600 5050
+Wire Wire Line
+	2400 5900 2600 5900
+Wire Wire Line
+	1100 5550 1550 5550
+Wire Wire Line
+	4800 4450 4800 5050
+Wire Wire Line
+	5650 4950 5650 5050
+Wire Wire Line
+	6050 4650 6050 5050
+Wire Wire Line
+	5700 3700 5700 4250
+Wire Wire Line
+	4800 2350 4800 2950
+Wire Wire Line
+	5650 2850 5650 2950
+Wire Wire Line
+	6050 2550 6050 2950
+Wire Wire Line
+	5700 1600 5700 2150
+Wire Wire Line
+	1500 2700 1500 2900
+Wire Wire Line
+	1250 1300 1400 1300
+Wire Wire Line
+	2250 1300 2400 1300
+Wire Wire Line
+	9650 4050 9650 4200
+Wire Wire Line
+	9550 4050 9550 4200
+Wire Wire Line
+	9450 1850 9450 2050
 $EndSCHEMATC

Commit message: Upraveno schéma a první, nepříliš povedená verze PCB.
Parts:
- removed D2: SM4007, Diode_SMD:D_MELF, symbol Diode:SM4007
- removed J2, J4: Screw_Terminal_01x01, symbol Connector:Screw_Terminal_01x01
- removed J7: M+, symbol Connector:Screw_Terminal_01x01
- removed J8: M-, symbol Connector:Screw_Terminal_01x01
- removed Q2: BUZ11, Package_TO_SOT_THT:TO-220-3_Vertical, symbol Transistor_FET:BUZ11
- removed R6: 470, symbol Device:R
- removed R7: 10k, symbol Device:R
- removed U3: LTV-817S, Package_DIP:SMDIP-4_W9.53mm, symbol Isolator:LTV-817S
- C1, C2: footprint (none) -> Capacitor_SMD:C_1206_3216Metric_Pad1.42x1.75mm_HandSolder
- DLed1, DLed2: footprint (none) -> LED_THT:LED_D3.0mm
- HC-SR4: renamed from HC-SR04; footprint (none) -> Connector_PinHeader_2.54mm:PinHeader_1x04_P2.54mm_Vertical
- J1, J3, J5, J6: footprint (none) -> TestPoint:TestPoint_Loop_D3.80mm_Drill2.5mm
- R1, R2, R3, R4, R5: footprint (none) -> Resistor_SMD:R_1206_3216Metric_Pad1.42x1.75mm_HandSolder
- SW1: footprint (none) -> Button_Switch_THT:SW_PUSH_6mm_H5mm
Connections:
- net labels removed: PWM2
- wire segments 78 -> 58

Commit message: Finální PCB k vytisknutí.
Changed lines of the file:
@@
 $EndDescr
-$Comp
-L MCU_Module:Arduino_Nano_v3.x A1
-U 1 1 5FC8165F
-P 9550 3050
-F 0 "A1" H 9550 1961 50  0000 C CNN
-F 1 "Arduino_Nano_v3.x" H 9550 1870 50  0000 C CNN
-F 2 "Module:Arduino_Nano" H 9550 3050 50  0001 C CIN
-F 3 "http://www.mouser.com/pdfdocs/Gravitech_Arduino_Nano3_0.pdf" H 9550 3050 50  0001 C CNN
-	1    9550 3050
-	1    0    0    -1
-$EndComp
 $Comp
 L Device:C C1
@@
 L power:GND #PWR0108
 U 1 1 5FC95D7A
-P 9650 4200
-F 0 "#PWR0108" H 9650 3950 50  0001 C CNN
-F 1 "GND" H 9655 4027 50  0000 C CNN
-F 2 "" H 9650 4200 50  0001 C CNN
-F 3 "" H 9650 4200 50  0001 C CNN
-	1    9650 4200
+P 9650 4400
+F 0 "#PWR0108" H 9650 4150 50  0001 C CNN
+F 1 "GND" H 9655 4227 50  0000 C CNN
+F 2 "" H 9650 4400 50  0001 C CNN
+F 3 "" H 9650 4400 50  0001 C CNN
+	1    9650 4400
 	1    0    0    -1
 $EndComp
@@
 L power:GND #PWR0109
 U 1 1 5FC9650E
-P 9550 4200
-F 0 "#PWR0109" H 9550 3950 50  0001 C CNN
-F 1 "GND" H 9555 4027 50  0000 C CNN
-F 2 "" H 9550 4200 50  0001 C CNN
-F 3 "" H 9550 4200 50  0001 C CNN
-	1    9550 4200
+P 9550 4400
+F 0 "#PWR0109" H 9550 4150 50  0001 C CNN
+F 1 "GND" H 9555 4227 50  0000 C CNN
+F 2 "" H 9550 4400 50  0001 C CNN
+F 3 "" H 9550 4400 50  0001 C CNN
+	1    9550 4400
 	1    0    0    -1
 $EndComp
@@
 L power:+5V #PWR0110
 U 1 1 5FC98089
-P 9450 1850
-F 0 "#PWR0110" H 9450 1700 50  0001 C CNN
-F 1 "+5V" H 9465 2023 50  0000 C CNN
-F 2 "" H 9450 1850 50  0001 C CNN
-F 3 "" H 9450 1850 50  0001 C CNN
-	1    9450 1850
-	1    0    0    -1
-$EndComp
-NoConn ~ 9650 2050
-NoConn ~ 9750 2050
-NoConn ~ 10050 2450
-NoConn ~ 10050 2550
-NoConn ~ 10050 2850
+P 9450 1600
+F 0 "#PWR0110" H 9450 1450 50  0001 C CNN
+F 1 "+5V" H 9465 1773 50  0000 C CNN
+F 2 "" H 9450 1600 50  0001 C CNN
+F 3 "" H 9450 1600 50  0001 C CNN
+	1    9450 1600
+	1    0    0    -1
+$EndComp
 $Comp
 L Connector:Conn_01x04_Female HC-SR4
@@
 Wire Wire Line
 	1400 3800 1150 3800
-Text GLabel 8900 2950 0    50   Input ~ 0
+Text GLabel 8500 2850 0    50   Input ~ 0
 Echo
-Text GLabel 8900 2850 0    50   Input ~ 0
+Text GLabel 8500 2750 0    50   Input ~ 0
 Trig
 $Comp
@@
 Wire Wire Line
 	4200 2150 4500 2150
-Wire Wire Line
-	9050 2950 8900 2950
-Text GLabel 8900 2650 0    50   Input ~ 0
+Text GLabel 8500 2550 0    50   Input ~ 0
 PWM1
-Wire Wire Line
-	8900 2850 9050 2850
 Text Notes 3650 800  0    50   ~ 0
 https://navody.arduino-shop.cz/navody-k-produktum/meric-vzdalenosti-ultrazvukovy.html
@@
 Wire Wire Line
 	1900 5050 2100 5050
-Text GLabel 8900 3450 0    50   Input ~ 0
+Text GLabel 8500 3350 0    50   Input ~ 0
 Led_yellow
-Text GLabel 8900 3550 0    50   Input ~ 0
+Text GLabel 8500 3450 0    50   Input ~ 0
 Led_green
-Wire Wire Line
-	8900 3450 9050 3450
-Wire Wire Line
-	9050 3550 8900 3550
 $Comp
 L Switch:SW_Push SW1
@@
 Wire Wire Line
 	2000 5550 2500 5550
-Text GLabel 8900 3350 0    50   Input ~ 0
+Text GLabel 8500 3250 0    50   Input ~ 0
 Btn1
-NoConn ~ 9050 2450
-NoConn ~ 9050 2550
-NoConn ~ 9050 3050
-NoConn ~ 9050 3150
-NoConn ~ 9050 3250
-NoConn ~ 9050 3750
-NoConn ~ 10050 3050
-NoConn ~ 10050 3150
-NoConn ~ 10050 3250
-NoConn ~ 10050 3350
-NoConn ~ 10050 3450
-NoConn ~ 10050 3550
-NoConn ~ 10050 3650
-NoConn ~ 10050 3750
 NoConn ~ 6350 2950
 Wire Wire Line
@@
 	1    0    0    -1
 $EndComp
-Wire Wire Line
-	8900 2650 9050 2650
 $Comp
 L power:+12V #PWR0105
@@
 Wire Wire Line
 	1500 2700 1500 2900
-Wire Wire Line
-	9650 4050 9650 4200
-Wire Wire Line
-	9550 4050 9550 4200
-Wire Wire Line
-	9450 1850 9450 2050
-NoConn ~ 9050 2750
-Wire Wire Line
-	8900 3350 9050 3350
+$Comp
+L MCU_Module:Arduino_Nano_v3.x A1
+U 1 1 5FC8165F
+P 9550 3050
+F 0 "A1" H 9550 1961 50  0000 C CNN
+F 1 "Arduino_Nano_v3.x" H 9550 1870 50  0000 C CNN
+F 2 "Module:Arduino_Nano" H 9550 3050 50  0001 C CIN
+F 3 "http://www.mouser.com/pdfdocs/Gravitech_Arduino_Nano3_0.pdf" H 9550 3050 50  0001 C CNN
+	1    9550 3050
+	1    0    0    -1
+$EndComp
+Wire Wire Line
+	8500 2550 9050 2550
+Wire Wire Line
+	8500 2750 9050 2750
+Wire Wire Line
+	8500 3250 9050 3250
+Wire Wire Line
+	8500 3350 9050 3350
+Wire Wire Line
+	9550 4050 9550 4400
+Wire Wire Line
+	9650 4050 9650 4400
+Wire Wire Line
+	9450 1600 9450 2050
+NoConn ~ 9750 2050
+NoConn ~ 9650 2050
+NoConn ~ 10050 2550
+NoConn ~ 10050 2450
+Wire Wire Line
+	8500 3450 9050 3450
+Wire Wire Line
+	8500 2850 9050 2850
+NoConn ~ 9050 2450
+NoConn ~ 9050 2650
+NoConn ~ 9050 2950
+NoConn ~ 9050 3050
+NoConn ~ 9050 3150
+NoConn ~ 9050 3550
 NoConn ~ 9050 3650
+NoConn ~ 9050 3750
+NoConn ~ 10050 3750
+NoConn ~ 10050 3650
+NoConn ~ 10050 3550
+NoConn ~ 10050 3450
+NoConn ~ 10050 3350
+NoConn ~ 10050 3250
+NoConn ~ 10050 3150
+NoConn ~ 10050 3050
+NoConn ~ 10050 2850
 $EndSCHEMATC

Commit message: Nová, zmenšená verze.
Changed lines of the file:
@@
-$EndComp
-$Comp
-L power:GND #PWR0108
-U 1 1 5FC95D7A
-P 9650 4400
-F 0 "#PWR0108" H 9650 4150 50  0001 C CNN
-F 1 "GND" H 9655 4227 50  0000 C CNN
-F 2 "" H 9650 4400 50  0001 C CNN
-F 3 "" H 9650 4400 50  0001 C CNN
-	1    9650 4400
-	1    0    0    -1
 $EndComp
 $Comp
@@
 Wire Wire Line
 	1400 3800 1150 3800
-Text GLabel 8500 2850 0    50   Input ~ 0
+Text GLabel 8500 2750 0    50   Input ~ 0
 Echo
-Text GLabel 8500 2750 0    50   Input ~ 0
+Text GLabel 8500 2950 0    50   Input ~ 0
 Trig
 $Comp
@@
 	9550 4050 9550 4400
 Wire Wire Line
-	9650 4050 9650 4400
-Wire Wire Line
 	9450 1600 9450 2050
 NoConn ~ 9750 2050
@@
 Wire Wire Line
 	8500 3450 9050 3450
-Wire Wire Line
-	8500 2850 9050 2850
 NoConn ~ 9050 2450
 NoConn ~ 9050 2650
-NoConn ~ 9050 2950
-NoConn ~ 9050 3050
 NoConn ~ 9050 3150
 NoConn ~ 9050 3550
@@
 NoConn ~ 10050 3050
 NoConn ~ 10050 2850
+Wire Wire Line
+	8500 2950 9050 2950
+NoConn ~ 9050 2850
+NoConn ~ 9650 4050
+$Comp
+L power:+5V #PWR?
+U 1 1 5FCEB636
+P 8500 3050
+F 0 "#PWR?" H 8500 2900 50  0001 C CNN
+F 1 "+5V" H 8515 3223 50  0000 C CNN
+F 2 "" H 8500 3050 50  0001 C CNN
+F 3 "" H 8500 3050 50  0001 C CNN
+	1    8500 3050
+	0    -1   -1   0
+$EndComp
+Wire Wire Line
+	8500 3050 9050 3050
 $EndSCHEMATC

Commit message: Verze s mosfet tranzistorem se neosvědčila. Nahrazeno relátkem.
Parts:
- removed D1: SM4007, Diode_SMD:D_MELF, symbol Diode:SM4007
- removed Q1: BUZ11, Package_TO_SOT_THT:TO-220-3_Vertical, symbol Transistor_FET:BUZ11
- removed R2, R5: 10k, Resistor_SMD:R_1206_3216Metric_Pad1.42x1.75mm_HandSolder, symbol Device:R
- removed SW1: SW_Push, Button_Switch_THT:SW_PUSH_6mm_H5mm, symbol Switch:SW_Push
- removed U2: LTV-817S, Package_DIP:SMDIP-4_W9.53mm, symbol Isolator:LTV-817S
- added K?: RSM822, Relay_THT:Relay_DPDT_Finder_40.52, symbol Relay:RSM822
- added Q?: BC817, Package_TO_SOT_SMD:SOT-23, symbol Transistor_BJT:BC817
- added R?: 10k, Resistor_SMD:R_1206_3216Metric_Pad1.42x1.75mm_HandSolder, symbol Device:R
- R1: value 470 -> 4k7
Connections:
- net labels removed: Btn1
- wire segments 58 -> 49
- no-connect marks 22 -> 23
Other:
- moved on the sheet: J5, J6, R1

Commit message: Změna pouzder pro kondíky.
Parts:
- C1, C2: footprint Capacitor_SMD:C_1206_3216Metric_Pad1.42x1.75mm_HandSolder -> Capacitor_THT:C_Disc_D3.0mm_W2.0mm_P2.50mm
- gave numbers to parts that had none: 3
- renumbered HC-SR4 to HC-SR1, J3 to J2, J5 to J3, J6 to J4
Connections:
- no-connect marks 23 -> 25
Changed lines of the file:
@@
 F 0 "C1" H 1115 2496 50  0000 L CNN
 F 1 "300n" H 1115 2405 50  0000 L CNN
-F 2 "Capacitor_SMD:C_1206_3216Metric_Pad1.42x1.75mm_HandSolder" H 1038 2300 50  0001 C CNN
+F 2 "Capacitor_THT:C_Disc_D3.0mm_W2.0mm_P2.50mm" H 1038 2300 50  0001 C CNN
 F 3 "~" H 1000 2450 50  0001 C CNN
 	1    1000 2450
@@
 F 0 "C2" H 2115 2496 50  0000 L CNN
 F 1 "100n" H 2115 2405 50  0000 L CNN
-F 2 "Capacitor_SMD:C_1206_3216Metric_Pad1.42x1.75mm_HandSolder" H 2038 2300 50  0001 C CNN
+F 2 "Capacitor_THT:C_Disc_D3.0mm_W2.0mm_P2.50mm" H 2038 2300 50  0001 C CNN
 F 3 "~" H 2000 2450 50  0001 C CNN
 	1    2000 2450
@@
 $EndComp
 $Comp
-L power:+5V #PWR0102
+L power:+5V #PWR08
 U 1 1 5FC87E3D
 P 2000 1900
-F 0 "#PWR0102" H 2000 1750 50  0001 C CNN
+F 0 "#PWR08" H 2000 1750 50  0001 C CNN
 F 1 "+5V" H 2015 2073 50  0000 C CNN
 F 2 "" H 2000 1900 50  0001 C CNN
@@
 $EndComp
 $Comp
-L power:+12V #PWR0103
+L power:+12V #PWR07
 U 1 1 5FC88135
 P 1000 1900
-F 0 "#PWR0103" H 1000 1750 50  0001 C CNN
+F 0 "#PWR07" H 1000 1750 50  0001 C CNN
 F 1 "+12V" H 1015 2073 50  0000 C CNN
 F 2 "" H 1000 1900 50  0001 C CNN
@@
 	2000 2100 2000 2300
 $Comp
-L power:GND #PWR0104
+L power:GND #PWR09
 U 1 1 5FC8917A
 P 1500 2900
-F 0 "#PWR0104" H 1500 2650 50  0001 C CNN
+F 0 "#PWR09" H 1500 2650 50  0001 C CNN
 F 1 "GND" H 1505 2727 50  0000 C CNN
 F 2 "" H 1500 2900 50  0001 C CNN
@@
 $EndComp
 $Comp
-L Connector:Screw_Terminal_01x01 J3
+L Connector:Screw_Terminal_01x01 J2
 U 1 1 5FC9259C
 P 2050 950
-F 0 "J3" H 1968 725 50  0000 C CNN
+F 0 "J2" H 1968 725 50  0000 C CNN
 F 1 "Screw_Terminal_01x01" H 1968 816 50  0000 C CNN
 F 2 "TestPoint:TestPoint_Loop_D3.80mm_Drill2.5mm" H 2050 950 50  0001 C CNN
@@
 $EndComp
 $Comp
-L power:GND #PWR0109
+L power:GND #PWR015
 U 1 1 5FC9650E
 P 9550 4400
-F 0 "#PWR0109" H 9550 4150 50  0001 C CNN
+F 0 "#PWR015" H 9550 4150 50  0001 C CNN
 F 1 "GND" H 9555 4227 50  0000 C CNN
 F 2 "" H 9550 4400 50  0001 C CNN
@@
 $EndComp
 $Comp
-L power:+5V #PWR0110
+L power:+5V #PWR06
 U 1 1 5FC98089
 P 9450 1600
-F 0 "#PWR0110" H 9450 1450 50  0001 C CNN
+F 0 "#PWR06" H 9450 1450 50  0001 C CNN
 F 1 "+5V" H 9465 1773 50  0000 C CNN
 F 2 "" H 9450 1600 50  0001 C CNN
@@
 $EndComp
 $Comp
-L Connector:Conn_01x04_Female HC-SR4
+L Connector:Conn_01x04_Female HC-SR1
 U 1 1 5FCA646F
 P 1600 3700
-F 0 "HC-SR4" H 1628 3676 50  0000 L CNN
+F 0 "HC-SR1" H 1628 3676 50  0000 L CNN
 F 1 "1-GND, 2-echo, 3-trig, 4-PWR (+5V)" H 1628 3585 50  0000 L CNN
 F 2 "Connector_PinHeader_2.54mm:PinHeader_1x04_P2.54mm_Vertical" H 1600 3700 50  0001 C CNN
@@
 $EndComp
 $Comp
-L power:GND #PWR0111
+L power:GND #PWR013
 U 1 1 5FCA6FD7
 P 1250 3600
-F 0 "#PWR0111" H 1250 3350 50  0001 C CNN
+F 0 "#PWR013" H 1250 3350 50  0001 C CNN
 F 1 "GND" V 1255 3472 50  0000 R CNN
 F 2 "" H 1250 3600 50  0001 C CNN
@@
 $EndComp
 $Comp
-L power:+5V #PWR0112
+L power:+5V #PWR014
 U 1 1 5FCA7540
 P 1250 3900
-F 0 "#PWR0112" H 1250 3750 50  0001 C CNN
+F 0 "#PWR014" H 1250 3750 50  0001 C CNN
 F 1 "+5V" V 1265 4028 50  0000 L CNN
 F 2 "" H 1250 3900 50  0001 C CNN
@@
 Trig
 $Comp
-L power:GND #PWR0116
+L power:GND #PWR010
 U 1 1 5FCC4DA2
 P 5650 3050
-F 0 "#PWR0116" H 5650 2800 50  0001 C CNN
+F 0 "#PWR010" H 5650 2800 50  0001 C CNN
 F 1 "GND" H 5655 2877 50  0000 C CNN
 F 2 "" H 5650 3050 50  0001 C CNN
@@
 $EndComp
 $Comp
-L power:GND #PWR0118
+L power:GND #PWR016
 U 1 1 5FCD0AF6
 P 2600 4600
-F 0 "#PWR0118" H 2600 4350 50  0001 C CNN
+F 0 "#PWR016" H 2600 4350 50  0001 C CNN
 F 1 "GND" H 2605 4427 50  0000 C CNN
 F 2 "" H 2600 4600 50  0001 C CNN
@@
 $EndComp
 $Comp
-L power:GND #PWR0119
+L power:GND #PWR017
 U 1 1 5FCD38A8
 P 2600 5050
-F 0 "#PWR0119" H 2600 4800 50  0001 C CNN
+F 0 "#PWR017" H 2600 4800 50  0001 C CNN
 F 1 "GND" H 2605 4877 50  0000 C CNN
 F 2 "" H 2600 5050 50  0001 C CNN
@@
 	1250 3600 1400 3600
 $Comp
-L Connector:Screw_Terminal_01x01 J5
+L Connector:Screw_Terminal_01x01 J3
 U 1 1 5FD0CD16
 P 7450 2450
-F 0 "J5" H 7368 2225 50  0000 C CNN
+F 0 "J3" H 7368 2225 50  0000 C CNN
 F 1 "M+" H 7368 2316 50  0000 C CNN
 F 2 "TestPoint:TestPoint_Loop_D3.80mm_Drill2.5mm" H 7450 2450 50  0001 C CNN
@@
 $EndComp
 $Comp
-L Connector:Screw_Terminal_01x01 J6
+L Connector:Screw_Terminal_01x01 J4
 U 1 1 5FD0DE67
 P 7450 2850
-F 0 "J6" H 7368 2625 50  0000 C CNN
+F 0 "J4" H 7368 2625 50  0000 C CNN
 F 1 "M-" H 7368 2716 50  0000 C CNN
 F 2 "TestPoint:TestPoint_Loop_D3.80mm_Drill2.5mm" H 7450 2850 50  0001 C CNN
@@
 $EndComp
 $Comp
-L power:+12V #PWR0105
+L power:+12V #PWR01
 U 1 1 5FCF4A8C
 P 1400 950
-F 0 "#PWR0105" H 1400 800 50  0001 C CNN
+F 0 "#PWR01" H 1400 800 50  0001 C CNN
 F 1 "+12V" V 1415 1078 50  0000 L CNN
 F 2 "" H 1400 950 50  0001 C CNN
@@
 $EndComp
 $Comp
-L power:GND #PWR0107
+L power:GND #PWR02
 U 1 1 5FCF4D70
 P 2400 950
-F 0 "#PWR0107" H 2400 700 50  0001 C CNN
+F 0 "#PWR02" H 2400 700 50  0001 C CNN
 F 1 "GND" V 2405 822 50  0000 R CNN
 F 2 "" H 2400 950 50  0001 C CNN
@@
 	1250 950  1300 950
 $Comp
-L power:PWR_FLAG #FLG0101
+L power:PWR_FLAG #FLG01
 U 1 1 5FCF95CF
 P 1300 950
-F 0 "#FLG0101" H 1300 1025 50  0001 C CNN
+F 0 "#FLG01" H 1300 1025 50  0001 C CNN
 F 1 "PWR_FLAG" H 1300 1123 50  0000 C CNN
 F 2 "" H 1300 950 50  0001 C CNN
@@
 	1300 950  1400 950
 $Comp
-L power:PWR_FLAG #FLG0104
+L power:PWR_FLAG #FLG02
 U 1 1 5FCFAF58
 P 2300 950
-F 0 "#FLG0104" H 2300 1025 50  0001 C CNN
+F 0 "#FLG02" H 2300 1025 50  0001 C CNN
 F 1 "PWR_FLAG" H 2300 1123 50  0000 C CNN
 F 2 "" H 2300 950 50  0001 C CNN
@@
 NoConn ~ 9050 3250
 $Comp
-L Transistor_BJT:BC817 Q?
+L Transistor_BJT:BC817 Q1
 U 1 1 5FD6B85F
 P 6000 2600
-F 0 "Q?" H 6191 2646 50  0000 L CNN
+F 0 "Q1" H 6191 2646 50  0000 L CNN
 F 1 "BC817" H 6191 2555 50  0000 L CNN
 F 2 "Package_TO_SOT_SMD:SOT-23" H 6200 2525 50  0001 L CIN
@@
 $EndComp
 $Comp
-L Relay:RSM822 K?
+L Relay:RSM822 K1
 U 1 1 5FD72A40
 P 6500 1900
-F 0 "K?" H 7130 1946 50  0000 L CNN
+F 0 "K1" H 7130 1946 50  0000 L CNN
 F 1 "RSM822" H 7130 1855 50  0000 L CNN
 F 2 "Relay_THT:Relay_DPDT_Finder_40.52" H 7850 1870 50  0001 C CNN
@@
 $EndComp
 $Comp
-L power:+12V #PWR?
+L power:+12V #PWR04
 U 1 1 5FD831EA
 P 6500 1450
-F 0 "#PWR?" H 6500 1300 50  0001 C CNN
+F 0 "#PWR04" H 6500 1300 50  0001 C CNN
 F 1 "+12V" V 6515 1578 50  0000 L CNN
 F 2 "" H 6500 1450 50  0001 C CNN
@@
 $EndComp
 $Comp
-L power:+12V #PWR?
+L power:+12V #PWR05
 U 1 1 5FD83A62
 P 6900 1450
-F 0 "#PWR?" H 6900 1300 50  0001 C CNN
+F 0 "#PWR05" H 6900 1300 50  0001 C CNN
 F 1 "+12V" V 6915 1578 50  0000 L CNN
 F 2 "" H 6900 1450 50  0001 C CNN
@@
 	7000 2450 6600 2450
 $Comp
-L power:GND #PWR?
+L power:GND #PWR012
 U 1 1 5FD86ED6
 P 7000 3050
-F 0 "#PWR?" H 7000 2800 50  0001 C CNN
+F 0 "#PWR012" H 7000 2800 50  0001 C CNN
 F 1 "GND" H 7005 2877 50  0000 C CNN
 F 2 "" H 7000 3050 50  0001 C CNN
@@
 	6100 2200 6100 2400
 $Comp
-L power:+12V #PWR?
+L power:+12V #PWR03
 U 1 1 5FD8968E
 P 6100 1450
-F 0 "#PWR?" H 6100 1300 50  0001 C CNN
+F 0 "#PWR03" H 6100 1300 50  0001 C CNN
 F 1 "+12V" V 6115 1578 50  0000 L CNN
 F 2 "" H 6100 1450 50  0001 C CNN
@@
 	6100 1450 6100 1600
 $Comp
-L power:GND #PWR?
+L power:GND #PWR011
 U 1 1 5FD8A380
 P 6100 3050
-F 0 "#PWR?" H 6100 2800 50  0001 C CNN
+F 0 "#PWR011" H 6100 2800 50  0001 C CNN
 F 1 "GND" H 6105 2877 50  0000 C CNN
 F 2 "" H 6100 3050 50  0001 C CNN
@@
 	6100 2800 6100 3050
 $Comp
-L Device:R R?
+L Device:R R2
 U 1 1 5FD8CC29
 P 5650 2800
-F 0 "R?" V 5443 2800 50  0000 C CNN
+F 0 "R2" V 5443 2800 50  0000 C CNN
 F 1 "10k" V 5534 2800 50  0000 C CNN
 F 2 "Resistor_SMD:R_1206_3216Metric_Pad1.42x1.75mm_HandSolder" V 5580 2800 50  0001 C CNN
@@
 Wire Wire Line
 	5650 2950 5650 3050
+NoConn ~ 6400 2200
+NoConn ~ 6800 2200
 $EndSCHEMATC
