File: osvitovka_pcb/osvitovka/osvitovka.sch (KiCad schematic (older format))
At the start: 20 parts, among them J1 Conn_01x05, J2 Conn_01x05, J3 Conn_01x04_Female, K1 RSM822, Q1 BC817, SW1 SW_Push, SW2 SW_Push, U1 L7805

Commit message: update
Parts:
- removed D2: LED, LED_THT:LED_D3.0mm, symbol Device:LED
- removed J1, J2: Conn_01x05, symbol Connector_Generic:Conn_01x05
- removed R2: 10k, Resistor_SMD:R_1206_3216Metric, symbol Device:R
- removed R6: 680, Resistor_SMD:R_1206_3216Metric, symbol Device:R
- removed SW2: SW_Push, Button_Switch_THT:SW_PUSH_6mm, symbol Switch:SW_Push
- added J1, J2: Conn_01x13_Female, Connector_PinSocket_2.54mm:PinSocket_1x13_P2.54mm_Vertical_SMD_Pin1Right, symbol Connector:Conn_01x13_Female
- J3: footprint (none) -> Connector_PinSocket_2.54mm:PinSocket_1x04_P2.54mm_Vertical
- K1: footprint Relay_THT:Relay_DPDT_Finder_40.52 -> Relay_THT:Relay_DPDT_Finder_30.22
- R1: footprint Resistor_SMD:R_1206_3216Metric -> Resistor_SMD:R_0805_2012Metric
- R2: renamed from R3; footprint Resistor_SMD:R_1206_3216Metric -> Resistor_SMD:R_0805_2012Metric
- R3: renamed from R4; footprint Resistor_SMD:R_1206_3216Metric -> Resistor_SMD:R_0805_2012Metric
- R4: renamed from R5; footprint Resistor_SMD:R_1206_3216Metric -> Resistor_SMD:R_0805_2012Metric
- renumbered D3 to D1, D1 to D2
Connections:
- wire segments 80 -> 102
- no-connect marks 0 -> 22
