File: osvitovka_ne555/osvitovkaNE555/osvitovkaNE555.kicad_pcb (KiCad board)
At the start: 2 copper layers, 19 parts, among them J1 +12V, J2 gnd, J3 Screw_Terminal_01x01, J4 Screw_Terminal_01x01, J5 Screw_Terminal_01x01, J6 Screw_Terminal_01x01, K1 RSM822, Q1 BC337, SW1 Start, SW2 Stop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

Commit message: další verze.
Parts:
- added J10: Conn_01x01_Male, Connector_Wire:SolderWirePad_1x01_Drill1.5mm, F.Cu at (193.0, 101.6)
- added J11: Conn_01x01_Male, Connector_Wire:SolderWirePad_1x01_Drill1.5mm, F.Cu at (205.7, 101.6)
- added J12: Conn_01x01_Male, Connector_Wire:SolderWirePad_1x01_Drill1.5mm, F.Cu at (218.4, 101.6)
- added J13: Conn_01x01_Male, Connector_Wire:SolderWirePad_1x01_Drill1.5mm, F.Cu at (110.5, 101.6)
- added J14: Conn_01x01_Male, Connector_Wire:SolderWirePad_1x01_Drill1.5mm, F.Cu at (123.2, 101.6)
- added J15: Conn_01x01_Male, Connector_Wire:SolderWirePad_1x01_Drill1.5mm, F.Cu at (135.9, 101.6)
- added J16: Conn_01x01_Male, Connector_Wire:SolderWirePad_1x01_Drill1.5mm, F.Cu at (148.6, 101.6)
- added J17: Conn_01x01_Male, Connector_Wire:SolderWirePad_1x01_Drill1.5mm, F.Cu at (161.3, 101.6)
- added J18: Conn_01x01_Male, Connector_Wire:SolderWirePad_1x01_Drill1.5mm, F.Cu at (174.0, 101.6)
- added J19: Conn_01x01_Male, Connector_Wire:SolderWirePad_1x01_Drill1.5mm, F.Cu at (186.7, 101.6)
- added J20: Conn_01x01_Male, Connector_Wire:SolderWirePad_1x01_Drill1.5mm, F.Cu at (199.4, 101.6)
- added J21: Conn_01x01_Male, Connector_Wire:SolderWirePad_1x01_Drill1.5mm, F.Cu at (212.1, 101.6)
- added J22: Conn_01x01_Male, Connector_Wire:SolderWirePad_1x01_Drill1.5mm, F.Cu at (224.8, 101.6)
- added J7: Conn_01x01_Male, Connector_Wire:SolderWirePad_1x01_Drill1.5mm, F.Cu at (154.9, 101.6)
- added J8: Conn_01x01_Male, Connector_Wire:SolderWirePad_1x01_Drill1.5mm, F.Cu at (167.6, 101.6)
- added J9: Conn_01x01_Male, Connector_Wire:SolderWirePad_1x01_Drill1.5mm, F.Cu at (180.3, 101.6)
- J3, J4, J5, J6: value Screw_Terminal_01x01 -> Conn_01x01_Male; footprint Connector_Wire:SolderWirePad_1x01_Drill1.2mm -> Connector_Wire:SolderWirePad_1x01_Drill1.5mm
- U1: footprint Package_DIP:DIP-8-16_W7.62mm_Socket -> Package_DIP:DIP-8_W7.62mm
- moved C1 131.1 mm to (170.2, 76.2), turned to 90 degrees
- moved SW2 118.3 mm to (203.2, 71.1)
- moved R4 112.4 mm to (151.1, 74.9), turned to 180 degrees
- moved R1 106.9 mm to (143.5, 72.4)
- moved C2 105.3 mm to (160.7, 62.2), turned to 180 degrees
- moved Q1 105.1 mm to (143.5, 57.8)
- moved SW1 101.8 mm to (184.2, 71.1)
- moved D1 98.8 mm to (127.6, 50.8)
- moved K1 96.4 mm to (136.5, 57.8), turned to 270 degrees
- moved R2 94.3 mm to (143.5, 77.5)
- moved R5 92.2 mm to (143.5, 69.8)
- moved R3 83.6 mm to (163.2, 55.9), turned to 180 degrees
- moved U1 83.4 mm to (155.6, 69.8)
- moved J5 68.1 mm to (129.5, 101.6)
- moved J6 51.1 mm to (142.2, 101.6)
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Connections:
- J4 pad 1: GND -> Net-(J3-Pad1)
- J5 pad 1: Net-(J5-Pad1) -> Net-(J3-Pad1)
- J6 pad 1: GND -> Net-(J3-Pad1)
- K1 pad 14: Net-(J3-Pad1) -> Net-(J10-Pad1)
- K1 pad 24: Net-(J5-Pad1) -> Net-(J3-Pad1)
Routing:
- net GND: track 0.00 -> 285.1 mm
- net +12V: track 0.00 -> 273.7 mm
- net Net-(J10-Pad1): track 0.00 -> 141.4 mm
- net Net-(J3-Pad1): track 0.00 -> 107.4 mm
- net Net-(R2-Pad2): track 0.00 -> 76.8 mm
- net Net-(R1-Pad2): track 0.00 -> 55.9 mm
- net Net-(C2-Pad1): track 0.00 -> 43.0 mm
- net Net-(Q1-Pad2): track 0.00 -> 21.3 mm
- net Net-(D1-Pad2): track 0.00 -> 14.5 mm
- net Net-(C1-Pad1): track 0.00 -> 7.51 mm
- net Net-(R4-Pad1): track 0.00 -> 4.44 mm

Commit message: update
Parts:
- added J23: Screw_Terminal_01x01, TestPoint:TestPoint_THTPad_D3.0mm_Drill1.5mm, F.Cu at (217.1, 48.2)
- added J24: Screw_Terminal_01x01, TestPoint:TestPoint_THTPad_D3.0mm_Drill1.5mm, F.Cu at (222.2, 43.2)
- added J25: Screw_Terminal_01x01, TestPoint:TestPoint_THTPad_D3.0mm_Drill1.5mm, F.Cu at (211.3, 58.3)
- added J26: Screw_Terminal_01x01, TestPoint:TestPoint_THTPad_D3.0mm_Drill1.5mm, F.Cu at (217.1, 53.3)
- added J27: Screw_Terminal_01x01, TestPoint:TestPoint_THTPad_D3.0mm_Drill1.5mm, F.Cu at (222.2, 48.2)
- added J28: Screw_Terminal_01x01, TestPoint:TestPoint_THTPad_D3.0mm_Drill1.5mm, F.Cu at (216.4, 58.3)
- added R6: 10k, Resistor_SMD:R_0805_2012Metric, B.Cu at (149.9, 47.0)
- C1: footprint Capacitor_THT:C_Disc_D10.0mm_W2.5mm_P5.00mm -> Capacitor_THT:C_Disc_D3.0mm_W1.6mm_P2.50mm
- D1: footprint Diode_THT:D_DO-41_SOD81_P10.16mm_Horizontal -> Diode_SMD:D_1206_3216Metric; moved to B.Cu
- J10, J11, J12, J13, J14, J15, J16, J17, J18, J19, J20, J21, J22, J3, J4, J5, J6, J7, J8, J9: value Conn_01x01_Male -> Screw_Terminal_01x01; footprint Connector_Wire:SolderWirePad_1x01_Drill1.5mm -> TestPoint:TestPoint_THTPad_D3.0mm_Drill1.5mm
- K1: footprint Relay_THT:Relay_DPDT_Finder_40.52 -> Relay_THT:Relay_DPDT_Finder_30.22
- Q1: footprint Package_TO_SOT_THT:TO-92_Inline -> Package_TO_SOT_SMD:SOT-23; moved to B.Cu
- R1: value 10k -> 420k; footprint Resistor_THT:R_Axial_DIN0204_L3.6mm_D1.6mm_P7.62mm_Horizontal -> Resistor_SMD:R_0805_2012Metric; moved to B.Cu
- R2: footprint Resistor_THT:R_Axial_DIN0204_L3.6mm_D1.6mm_P7.62mm_Horizontal -> Resistor_SMD:R_0805_2012Metric; moved to B.Cu
- R3: value 470k-1M -> 10k; footprint Resistor_THT:R_Axial_DIN0204_L3.6mm_D1.6mm_P7.62mm_Horizontal -> Resistor_SMD:R_0805_2012Metric; moved to B.Cu
- R4: value 4k7 -> 50k; footprint Resistor_THT:R_Axial_DIN0204_L3.6mm_D1.6mm_P7.62mm_Horizontal -> Potentiometer_THT:Potentiometer_Runtron_RM-063_Horizontal; moved to B.Cu
- R5: value 10k -> 4k7; footprint Resistor_THT:R_Axial_DIN0204_L3.6mm_D1.6mm_P7.62mm_Horizontal -> Resistor_SMD:R_0805_2012Metric; moved to B.Cu
- U1: value NE555 -> LMC555xN
- moved J3 122.7 mm to (212.1, 43.2)
- moved J13 103.5 mm to (202.0, 53.3)
- moved J14 99.4 mm to (207.0, 48.2)
- moved J6 83.6 mm to (202.0, 43.2)
- moved J4 83.5 mm to (186.1, 54.9)
- moved J16 75.8 mm to (196.9, 43.2)
- moved J15 74.2 mm to (196.2, 58.3)
- moved J5 70.2 mm to (186.1, 60.0)
- moved J7 67.9 mm to (196.9, 48.2)
- moved J20 61.1 mm to (217.1, 43.2)
- moved J19 59.1 mm to (212.1, 48.2)
- moved J17 58.9 mm to (201.2, 58.3)
- moved J18 58.5 mm to (207.0, 53.3)
- moved J11 58.4 mm to (207.0, 43.2)
- moved J9 57.6 mm to (202.0, 48.2)
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Connections:
- J11 pad 1: Net-(J10-Pad1) -> GND
- J14 pad 1: GND -> Net-(J10-Pad1)
- J16 pad 1: GND -> Net-(J10-Pad1)
- J18 pad 1: GND -> Net-(J18-Pad1)
- J20 pad 1: GND -> Net-(J18-Pad1)
- J22 pad 1: GND -> Net-(J18-Pad1)
- J3 pad 1: Net-(J3-Pad1) -> GND
- J4 pad 1: Net-(J3-Pad1) -> Net-(J10-Pad1)
- J5 pad 1: Net-(J3-Pad1) -> GND
- J6 pad 1: Net-(J3-Pad1) -> Net-(J10-Pad1)
- J7 pad 1: Net-(J3-Pad1) -> GND
- J9 pad 1: Net-(J10-Pad1) -> GND
- K1 pad 24: Net-(J3-Pad1) -> Net-(J18-Pad1)
- R3 pad 2: Net-(C2-Pad1) -> Net-(R3-Pad2)
- R4 pad 1: Net-(R4-Pad1) -> Net-(R1-Pad2)
- R4 pad 2: Net-(Q1-Pad2) -> Net-(C2-Pad1)
- R5 pad 1: Net-(Q1-Pad2) -> Net-(R5-Pad1)
- R5 pad 2: GND -> Net-(Q1-Pad2)
- SW1 pad 2: Net-(R1-Pad2) -> Net-(R2-Pad2)
- SW2 pad 2: Net-(R2-Pad2) -> Net-(R3-Pad2)
- U1 pad 2: Net-(R1-Pad2) -> Net-(R2-Pad2)
- U1 pad 3: Net-(R4-Pad1) -> Net-(R5-Pad1)
- U1 pad 4: Net-(R2-Pad2) -> Net-(R3-Pad2)
Routing:
- net GND: track 285.1 -> 0.11 mm
- net +12V: track 273.7 -> 0.45 mm
- net Net-(J10-Pad1): track 141.4 -> 0.00 mm
- net Net-(J3-Pad1): track 107.4 -> 0.00 mm
- net Net-(R2-Pad2): track 76.8 -> 0.00 mm
- net Net-(R1-Pad2): track 55.9 -> 0.00 mm
- net Net-(C2-Pad1): track 43.0 -> 0.00 mm
- net Net-(Q1-Pad2): track 21.3 -> 0.00 mm
- net Net-(D1-Pad2): track 14.5 -> 0.00 mm
- net Net-(C1-Pad1): track 7.51 -> 0.00 mm
- net Net-(R4-Pad1): track 4.44 -> 0.00 mm

Commit message: finální verze pro výrobu č. 1
Parts:
- removed SW2: Stop, Button_Switch_THT:SW_PUSH_6mm_H8mm
- moved J3 155.5 mm to (70.5, 107.3)
- moved J6 131.8 mm to (86.8, 107.3)
- moved J4 122.0 mm to (75.9, 107.3)
- moved J7 120.2 mm to (92.2, 107.3)
- moved J9 115.2 mm to (103.1, 107.3)
- moved J5 114.9 mm to (81.4, 107.3)
- moved J11 113.0 mm to (114.0, 107.3)
- moved J8 107.2 mm to (97.7, 107.3)
- moved J10 103.6 mm to (108.5, 107.3)
- moved J14 96.9 mm to (130.3, 107.3)
- moved J13 94.2 mm to (124.8, 107.3)
- moved J12 85.9 mm to (119.4, 107.3)
- moved J16 85.0 mm to (141.1, 107.3)
- moved J20 84.0 mm to (162.9, 107.3)
- moved J19 80.5 mm to (157.5, 107.3)
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Routing:
- net GND: track 0.11 -> 414.8 mm
- net Net-(J18-Pad1): track 0.00 -> 144.1 mm
- net Net-(J10-Pad1): track 0.00 -> 105.2 mm
- net +12V: track 0.45 -> 92.1 mm
- net Net-(R2-Pad2): track 0.00 -> 64.7 mm
- net Net-(C2-Pad1): track 0.00 -> 30.3 mm
- net Net-(D1-Pad2): track 0.00 -> 30.1 mm
- net Net-(Q1-Pad2): track 0.00 -> 12.8 mm
- net Net-(C1-Pad1): track 0.00 -> 6.73 mm
- net Net-(R1-Pad2): track 0.00 -> 6.33 mm
- net Net-(R3-Pad2): track 0.00 -> 3.51 mm
- net Net-(R5-Pad1): track 0.00 -> 3.41 mm
- added copper zone on B.Cu, net GND
Other:
- board text added: "+12V"

Commit message: test a upgrade pcb.
Parts:
- Q1: value BC337 -> BC817
- turned Q1 to 180 degrees
Connections:
- Q1 pad 1: Net-(D1-Pad2) -> Net-(Q1-Pad1)
- Q1 pad 2: Net-(Q1-Pad2) -> GND
- Q1 pad 3: GND -> Net-(D1-Pad2)
- R5 pad 2: Net-(Q1-Pad2) -> Net-(Q1-Pad1)
- R6 pad 1: Net-(Q1-Pad2) -> Net-(Q1-Pad1)
Routing:
- net Net-(Q1-Pad1): track 0.00 -> 12.9 mm
- net Net-(Q1-Pad2): track 12.8 -> 0.00 mm
- net GND: track 414.8 -> 415.7 mm
