File: osvitovka_ne555/osvitovkaNE555/osvitovkaNE555.sch (KiCad schematic (older format))
At the start: 19 parts, among them J1 +12V, J2 gnd, J3 Screw_Terminal_01x01, J4 Screw_Terminal_01x01, J5 Screw_Terminal_01x01, J6 Screw_Terminal_01x01, K1 RSM822, Q1 BC337, SW1 Start, SW2 Stop, U1 NE555

Commit message: další verze.
Parts:
- removed J3, J4, J5, J6: Screw_Terminal_01x01, Connector_Wire:SolderWirePad_1x01_Drill1.2mm, symbol Connector:Screw_Terminal_01x01
- added J10, J11, J12, J13, J14, J15, J16, J17, J18, J19, J20, J21, J22, J3, J4, J5, J6, J7, J8, J9: Conn_01x01_Male, Connector_Wire:SolderWirePad_1x01_Drill1.5mm, symbol Connector:Conn_01x01_Male
Connections:
- wire segments 60 -> 98

Commit message: update
Parts:
- removed J10, J11, J12, J13, J14, J15, J16, J17, J18, J19, J20, J21, J22, J3, J4, J5, J6, J7, J8, J9: Conn_01x01_Male, Connector_Wire:SolderWirePad_1x01_Drill1.5mm, symbol Connector:Conn_01x01_Male
- removed U1: NE555, Package_DIP:DIP-8_W7.62mm, symbol Timer:NE555
- added J10, J11, J12, J13, J14, J15, J16, J17, J18, J19, J20, J21, J22, J23, J24, J25, J26, J27, J28, J3, J4, J5, J6, J7, J8, J9: Screw_Terminal_01x01, TestPoint:TestPoint_THTPad_D3.0mm_Drill1.5mm, symbol Connector:Screw_Terminal_01x01
- added R4: 50k, Potentiometer_THT:Potentiometer_Runtron_RM-063_Horizontal, symbol Device:RTRIM
- added U1: LMC555xN, Package_DIP:DIP-8_W7.62mm, symbol Timer:LMC555xN
- C1: footprint Capacitor_THT:C_Disc_D10.0mm_W2.5mm_P5.00mm -> Capacitor_THT:C_Disc_D3.0mm_W1.6mm_P2.50mm
- D1: footprint Diode_THT:D_DO-41_SOD81_P10.16mm_Horizontal -> Diode_SMD:D_1206_3216Metric
- K1: footprint Relay_THT:Relay_DPDT_Finder_40.52 -> Relay_THT:Relay_DPDT_Finder_30.22
- Q1: footprint Package_TO_SOT_THT:TO-92_Inline -> Package_TO_SOT_SMD:SOT-23
- R1: renamed from R3; value 470k-1M -> 420k; footprint Resistor_THT:R_Axial_DIN0204_L3.6mm_D1.6mm_P7.62mm_Horizontal -> Resistor_SMD:R_0805_2012Metric
- R2: renamed from R1; footprint Resistor_THT:R_Axial_DIN0204_L3.6mm_D1.6mm_P7.62mm_Horizontal -> Resistor_SMD:R_0805_2012Metric
- R3: renamed from R2; footprint Resistor_THT:R_Axial_DIN0204_L3.6mm_D1.6mm_P7.62mm_Horizontal -> Resistor_SMD:R_0805_2012Metric
- R5: renamed from R4; footprint Resistor_THT:R_Axial_DIN0204_L3.6mm_D1.6mm_P7.62mm_Horizontal -> Resistor_SMD:R_0805_2012Metric
- R6: renamed from R5; footprint Resistor_THT:R_Axial_DIN0204_L3.6mm_D1.6mm_P7.62mm_Horizontal -> Resistor_SMD:R_0805_2012Metric
Connections:
- wire segments 98 -> 111
Other:
- moved on the sheet: R1

Commit message: finální verze pro výrobu č. 1
Parts:
- removed SW2: Stop, Button_Switch_THT:SW_PUSH_6mm_H8mm, symbol Switch:SW_Push
Changed lines of the file:
@@
-$EndComp
-$Comp
-L Switch:SW_Push SW2
-U 1 1 5FD01299
-P 3750 4300
-F 0 "SW2" V 3796 4252 50  0000 R CNN
-F 1 "Stop" V 3705 4252 50  0000 R CNN
-F 2 "Button_Switch_THT:SW_PUSH_6mm_H8mm" H 3750 4500 50  0001 C CNN
-F 3 "~" H 3750 4500 50  0001 C CNN
-	1    3750 4300
-	0    -1   -1   0
 $EndComp
 $Comp
@@
 Wire Wire Line
 	3050 2000 3750 2000
-Wire Wire Line
-	3050 4750 3750 4750
 Connection ~ 5600 4750
 Wire Wire Line
@@
 Wire Wire Line
 	3750 2850 3750 3750
-Wire Wire Line
-	3750 4500 3750 4750
-Connection ~ 3750 4750
-Connection ~ 3750 3750
-Wire Wire Line
-	3750 3750 3750 4100
 Wire Wire Line
 	4950 3150 4950 2000
@@
 Wire Wire Line
 	2100 2100 2300 2100
-Wire Wire Line
-	3750 4750 4350 4750
 Connection ~ 4350 4750
 Wire Wire Line
@@
 	5600 3050 5600 3550
 Connection ~ 5600 3550
+Wire Wire Line
+	3050 4750 4350 4750
 $EndSCHEMATC

Commit message: test a upgrade pcb.
Parts:
- removed Q1: BC337, Package_TO_SOT_SMD:SOT-23, symbol Transistor_BJT:BC337
- added Q1: BC817, Package_TO_SOT_SMD:SOT-23, symbol Transistor_BJT:BC817
Connections:
- net GND: now also Q1.2 (E)
- net at R5.2, R6.1: now also Q1.1 (B)
- net at D1.2 (A), K1.A1: now also Q1.3 (C)
Changed lines of the file:
@@
-$EndComp
-$Comp
-L Transistor_BJT:BC337 Q1
-U 1 1 5FCFC78D
-P 7200 3350
-F 0 "Q1" H 7391 3396 50  0000 L CNN
-F 1 "BC337" H 7391 3305 50  0000 L CNN
-F 2 "Package_TO_SOT_SMD:SOT-23" H 7400 3275 50  0001 L CIN
-F 3 "https://diotec.com/tl_files/diotec/files/pdf/datasheets/bc337.pdf" H 7200 3350 50  0001 L CNN
-	1    7200 3350
-	1    0    0    -1
 $EndComp
 $Comp
@@
 Wire Wire Line
 	3050 4750 4350 4750
+$Comp
+L Transistor_BJT:BC817 Q1
+U 1 1 5FDE9E5B
+P 7200 3350
+F 0 "Q1" H 7391 3396 50  0000 L CNN
+F 1 "BC817" H 7391 3305 50  0000 L CNN
+F 2 "Package_TO_SOT_SMD:SOT-23" H 7400 3275 50  0001 L CIN
+F 3 "http://www.fairchildsemi.com/ds/BC/BC817.pdf" H 7200 3350 50  0001 L CNN
+	1    7200 3350
+	1    0    0    -1
+$EndComp
 $EndSCHEMATC
