File: pipatko/Pipatko/Pipatko.kicad_pcb (KiCad board)
At the start: 2 copper layers, 15 parts, among them J1 hroty, J2 vypinac, J3 9V= 1+ / 2-, Q1 BC547, Q2 BC557, SW1 test tlacitko

Commit message: První verze PCB.
Parts:
- removed SW1: test tlacitko, LPouzdra:AR_SW_PUSH_6mm
- J2: footprint Connector_Phoenix_MC_HighVoltage:PhoenixContact_MCV_1,5_2-G-5.08_1x02_P5.08mm_Vertical -> LPouzdra:AR_PinHeader_1x02_P2.54mm_Vertical
- R4: moved to B.Cu
- moved J1 49.5 mm to (104.6, 80.8), turned to 270 degrees
- moved Q2 31.0 mm to (138.7, 87.1)
- moved D1 30.2 mm to (144.8, 90.9), turned to 90 degrees
- moved R2 28.1 mm to (135.4, 80.8), turned to 270 degrees
- moved J2 26.7 mm to (123.2, 100.6)
- moved R4 26.4 mm to (108.2, 93.7), turned to 270 degrees
- moved R1 25.0 mm to (104.6, 93.7), turned to 270 degrees
- moved J3 24.7 mm to (128.8, 101.6)
- moved R3 24.5 mm to (118.1, 102.4)
- moved R5 17.4 mm to (131.3, 80.8), turned to 270 degrees
- moved C1 17.0 mm to (144.8, 93.7), turned to 270 degrees
- moved Q1 14.0 mm to (146.1, 102.4), turned to 180 degrees
- moved D2 12.7 mm to (139.4, 105.7), turned to 90 degrees
- moved BZ1 8.52 mm to (120.1, 90.7), turned to 90 degrees
Connections:
- net Net-(D2-Pad2) renamed GND
Routing:
- net Net-(C1-Pad1): track 0.00 -> 57.4 mm
- net GND: track 0.00 -> 52.1 mm
- net Net-(C1-Pad2): track 0.00 -> 51.4 mm
- net Net-(BZ1-Pad2): track 0.00 -> 51.0 mm
- net Net-(D1-Pad1): track 0.00 -> 24.5 mm
- net Net-(BZ1-Pad1): track 0.00 -> 21.2 mm
- net Net-(R3-Pad3): track 0.00 -> 12.6 mm
- net Net-(Q2-Pad2): track 0.00 -> 10.3 mm
- net Net-(J1-Pad2): track 0.00 -> 7.87 mm
- net Net-(J2-Pad2): track 0.00 -> 6.22 mm
- added copper zone on B.Cu, net GND
Other:
- board text added: "+"
