File: studium/tranzistoryJakoSpinace/tranzistoryJakoSpinace.kicad_pcb (KiCad board)
At the start: 2 copper layers, 23 parts, among them J1 Conn_01x02_Male, J2 Conn_01x02_Male, J3 Conn_01x02_Male, Q1 BC807, Q2 BC817, Q3 BC817

Commit message: skorofinální verze.
Parts:
- moved TP3 70.0 mm to (104.9, 116.6)
- moved J3 64.5 mm to (93.2, 147.1), turned to 270 degrees
- moved TP6 62.0 mm to (108.0, 127.8)
- moved TP5 61.2 mm to (101.9, 127.8)
- moved R5 59.0 mm to (104.9, 147.1), turned to 180 degrees
- moved TP1 54.8 mm to (110.7, 140.7)
- moved TP9 52.7 mm to (113.8, 151.6)
- moved R6 52.7 mm to (121.4, 148.3), turned to 270 degrees
- moved TP8 50.2 mm to (107.7, 151.6)
- moved TP4 46.4 mm to (122.9, 116.6)
- moved TP7 38.5 mm to (126.0, 127.8)
- moved R4 38.5 mm to (135.9, 122.2), turned to 270 degrees
- moved TP2 38.3 mm to (119.9, 127.8)
- moved Q3 31.4 mm to (110.7, 146.3), turned to 90 degrees
- moved D2 31.1 mm to (121.4, 153.7), turned to 90 degrees
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Routing:
- net +12V: track 0.00 -> 161.3 mm
- net GND: track 0.00 -> 96.2 mm
- net Net-(Q2-Pad3): track 0.00 -> 19.6 mm
- net Net-(Q1-Pad3): track 0.00 -> 17.6 mm
- net Net-(Q3-Pad2): track 0.00 -> 14.0 mm
- net (no net): track 0.00 -> 13.7 mm
- net Net-(Q1-Pad1): track 0.00 -> 12.1 mm
- net Net-(J3-Pad1): track 0.00 -> 10.7 mm
- net Net-(Q3-Pad1): track 0.00 -> 8.54 mm
- net Net-(Q2-Pad1): track 0.00 -> 7.78 mm
- net Net-(J2-Pad1): track 0.00 -> 5.33 mm
- net Net-(D1-Pad2): track 0.00 -> 3.08 mm
- net Net-(D2-Pad2): track 0.00 -> 2.82 mm
- added copper zone on F.Cu, net GND
Other:
- board text added: "+"
- board text added: "-"
- board text added: "B"
- board text added: "C"
- board text added: "E"
- board text added: "NPN"
- board text added: "PNP"

Commit message: finální verze.
Routing:
- net GND: track 96.2 -> 37.0 mm
Other:
- board text added: "http://robodoupe.cz/ 2012/ peckovy-tranzistor/"
Changed lines of the file:
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@@
   (general
     (thickness 1.6)
-    (drawings 14)
-    (tracks 85)
+    (drawings 15)
+    (tracks 79)
     (zones 0)
     (modules 23)
@@
     )
   )
+  (gr_text "http://robodoupe.cz/\n2012/\npeckovy-tranzistor/" (at 132.842 144.78 90) (layer F.Cu)
+    (effects (font (size 1.55 1.3) (thickness 0.325)))
+  )
   (gr_text - (at 90.678 130.556 90) (layer F.Cu)
     (effects (font (size 1.5 1.5) (thickness 0.3)))
@@
   (segment (start 92.202 120.65) (end 94.996 120.65) (width 0.508) (layer F.Cu) (net 0))
   (segment (start 135.89 123.199) (end 135.89 126.2745) (width 0.508) (layer F.Cu) (net 1))
-  (segment (start 134.5835 155.1575) (end 135.89 153.851) (width 0.508) (layer F.Cu) (net 2))
   (segment (start 135.89 130.556) (end 135.89 130.048) (width 0.508) (layer F.Cu) (net 2))
   (segment (start 135.89 130.048) (end 135.89 129.2495) (width 0.508) (layer F.Cu) (net 2))
   (segment (start 135.89 131.826) (end 135.89 130.048) (width 0.508) (layer F.Cu) (net 2))
-  (segment (start 121.412 155.1575) (end 134.5835 155.1575) (width 0.508) (layer F.Cu) (net 2))
-  (segment (start 135.636 133.096) (end 135.89 133.35) (width 0.508) (layer F.Cu) (net 2))
-  (segment (start 135.89 153.851) (end 135.89 133.35) (width 0.508) (layer F.Cu) (net 2))
-  (segment (start 135.89 133.35) (end 135.89 131.826) (width 0.508) (layer F.Cu) (net 2))
-  (segment (start 113.792 133.096) (end 135.636 133.096) (width 0.508) (layer F.Cu) (net 2))
   (segment (start 107.95 127.762) (end 107.95 130.27) (width 0.508) (layer F.Cu) (net 2))
   (segment (start 90.678 133.096) (end 107.95 133.096) (width 0.508) (layer F.Cu) (net 2))
