File: logicAnalyzerAdapter/LAAdapter/LAAdapter.sch (KiCad schematic (older format))
At the start: 1 part, among them J1 Conn_02x05_Counter_Clockwise

Commit message: prvni verze s PCB
Parts:
- added H1, H2, H3, H4: MountingHole, MountingHole:MountingHole_3.5mm_Pad, symbol Mechanical:MountingHole
- added J2, J3: Conn_02x10_Counter_Clockwise, AR_Library:AR_PinHeader_2x10_P2.54mm_Vertical, symbol Connector_Generic:Conn_02x10_Counter_Clockwise
- added J5, J6: Conn_01x01_Female, AR_Library:AR_AMASS_4mm_Horizontal, symbol Connector:Conn_01x01_Female
- J1: footprint (none) -> AR_Library:AR_PinHeader_2x05_P2.54mm_Horizontal
Connections:
- wire segments 0 -> 128
Other:
- moved on the sheet: J1

Commit message: verze 2.0 s PCB, zjednodušená
Parts:
- removed H1, H2, H3, H4: MountingHole, MountingHole:MountingHole_3.5mm_Pad, symbol Mechanical:MountingHole
- removed J2, J3: Conn_02x10_Counter_Clockwise, AR_Library:AR_PinHeader_2x10_P2.54mm_Vertical, symbol Connector_Generic:Conn_02x10_Counter_Clockwise
- added J2: Conn_02x02_Odd_Even, AR_Library:AR_PinHeader_2x02_P2.54mm_Vertical, symbol Connector_Generic:Conn_02x02_Odd_Even
- added TP1, TP2, TP3, TP4, TP5, TP6, TP7: TestPoint, AR_Library:AR_PinHeader_1x01_P2.54mm_Vertical, symbol Connector:TestPoint
- renumbered J5 to J3, J6 to J4
Connections:
- wire segments 128 -> 24
Other:
- moved on the sheet: J1, J3, J4
