File: logicAnalyzerAdapter/LAAdapter/LAAdapter.kicad_pcb (KiCad board)
At the start: 2 copper layers, 9 parts, among them J1 Conn_02x05_Counter_Clockwise, J2 Conn_02x10_Counter_Clockwise, J3 Conn_02x10_Counter_Clockwise, J5 Conn_01x01_Female, J6 Conn_01x01_Female

Commit message: verze 2.0 s PCB, zjednodušená
Parts:
- removed H1, H2, H3, H4: MountingHole, MountingHole:MountingHole_3.5mm_Pad
- removed the J3 at (200.7, 52.1)
- added TP1: TestPoint, AR_Library:AR_PinHeader_1x01_P2.54mm_Vertical, F.Cu at (186.7, 58.4)
- added TP2: TestPoint, AR_Library:AR_PinHeader_1x01_P2.54mm_Vertical, F.Cu at (177.8, 58.4)
- added TP3: TestPoint, AR_Library:AR_PinHeader_1x01_P2.54mm_Vertical, F.Cu at (177.8, 54.0)
- added TP4: TestPoint, AR_Library:AR_PinHeader_1x01_P2.54mm_Vertical, F.Cu at (177.8, 62.9)
- added TP5: TestPoint, AR_Library:AR_PinHeader_1x01_P2.54mm_Vertical, F.Cu at (177.8, 71.8)
- added TP6: TestPoint, AR_Library:AR_PinHeader_1x01_P2.54mm_Vertical, F.Cu at (186.7, 67.3)
- added TP7: TestPoint, AR_Library:AR_PinHeader_1x01_P2.54mm_Vertical, F.Cu at (177.8, 67.3)
- J2: value Conn_02x10_Counter_Clockwise -> Conn_02x02_Odd_Even; footprint AR_Library:AR_PinHeader_2x10_P2.54mm_Vertical -> AR_Library:AR_PinHeader_2x02_P2.54mm_Vertical; moved to F.Cu
- moved J2 28.8 mm to (196.8, 52.1), turned to 0 degrees
- moved J1 5.12 mm to (170.2, 57.8)
- moved J3 1.80 mm to (212.1, 72.4)
- moved J4 1.80 mm to (212.1, 53.3)
- renumbered J5 to J3, J6 to J4
Connections:
- J2 pad 1: Net-(J1-Pad10) -> Net-(J1-Pad2)
- J2 pad 2: Net-(J2-Pad10) -> Net-(J2-Pad2)
- J2 pad 3: Net-(J1-Pad9) -> Net-(J1-Pad10)
- J2 pad 4: Net-(J2-Pad10) -> Net-(J2-Pad2)
- J3 pad 1: Net-(J2-Pad10) -> Net-(J1-Pad4)
- J4 pad 1: Net-(J3-Pad10) -> Net-(J2-Pad2)
Routing:
- net Net-(J1-Pad4): track 52.1 -> 102.4 mm, vias 2 -> 0
- net Net-(J2-Pad10): track 42.4 -> 0.00 mm
- net Net-(J3-Pad10): track 40.6 -> 0.00 mm
- net Net-(J1-Pad10): track 30.5 -> 51.4 mm, vias 2 -> 0
- net Net-(J1-Pad7): track 26.7 -> 8.41 mm, vias 2 -> 0
- net Net-(J1-Pad5): track 25.4 -> 7.62 mm, vias 2 -> 0
- net Net-(J1-Pad9): track 26.7 -> 9.20 mm, vias 2 -> 0
- net Net-(J1-Pad3): track 25.4 -> 8.41 mm, vias 2 -> 0
- net Net-(J1-Pad1): track 25.4 -> 9.20 mm, vias 2 -> 0
- net Net-(J2-Pad2): track 0.00 -> 15.2 mm
- net Net-(J1-Pad8): track 47.0 -> 39.0 mm, vias 2 -> 0
- net Net-(J1-Pad6): track 64.8 -> 58.0 mm, vias 2 -> 0
- net Net-(J1-Pad2): track 30.5 -> 32.7 mm, vias 2 -> 0

Commit message: update součástky v knihovně, update pcb
Parts:
- J3, J4: moved to F.Cu
- moved J3 0.63 mm to (211.5, 72.4), turned to 270 degrees
- moved J4 0.63 mm to (211.5, 53.3), turned to 270 degrees
